File: SDB628_Modul_3.kicad_pcb (KiCad board)
At the start: 2 copper layers, 45.2 x 27.7 mm, 21 parts, among them J1 Batt_In, J2 +15V_ON_OFF?, J3 Pow_Out_5V, J4 Pow_Out_15V, J5 BR1_1, J6 BR1_2, Q1 BSS123, Q2 AO3407, U1 DC-DC-SDB628, U2 DC-DC-SDB628

Commit message: Add files via upload
Parts:
- removed REF** (x2): MH_M2, MountingHole:MountingHole_2.2mm_M2
- added 1: MH_M2, MountingHole:MountingHole_2.2mm_M2, F.Cu at (81.5, 34.8)
- added 2: MH_M2, MountingHole:MountingHole_2.2mm_M2, F.Cu at (81.3, 56.4)
- C1, C2, F1, F2, R1, R2, R3: moved to F.Cu
- J2: value +15V_ON_OFF? -> Ubat_PowUce
- moved R1 5.09 mm to (102.6, 53.3)
- moved J3 4.33 mm to (120.7, 40.4), turned to 0 degrees
- moved R3 2.30 mm to (80.5, 46.5)
- moved F1 2.17 mm to (87.1, 46.0)
- moved F2 1.72 mm to (92.5, 38.9), turned to -90 degrees
- moved R2 1.69 mm to (89.7, 46.0)
- moved J4 0.77 mm to (120.7, 48.0)
- moved J1 0.76 mm to (83.6, 39.6)
- moved C1 0.76 mm to (102.9, 37.3)
- moved Q2 0.72 mm to (93.5, 45.5)
- moved 4 0.36 mm to (120.4, 56.1)
- moved J2 0.36 mm to (83.8, 48.2)
- moved Q1 0.25 mm to (100.1, 44.7)
- moved 3 0.25 mm to (120.7, 35.1)
- renumbered REF** to 3, REF** to 4
Routing:
- net GND: track 172.8 -> 135.3 mm
- net Net-(F1-Pad1): track 16.8 -> 5.88 mm
- net Net-(C2-Pad1): track 20.2 -> 11.1 mm
- net Net-(C1-Pad1): track 14.7 -> 9.09 mm
- net Net-(J2-Pad2): track 27.3 -> 28.8 mm
- net Net-(Q1-Pad3): track 13.1 -> 11.8 mm
- net Net-(J3-Pad2): track 8.78 -> 7.57 mm
- net Net-(J4-Pad2): track 10.7 -> 9.98 mm
- net Net-(J2-Pad1): track 4.06 -> 3.39 mm
Other:
- board text added: "pin_POW_UCE"
- board text added: "pin_UBAT"
- board text removed: "pin_E_NEG"
- board text removed: "pin_E_POS"
